Commit message: fixed something

File: resources/robots/a1/urdf/a1.urdf (robot description, URDF)
Before this commit: robot a1_description, 23 links, 22 joints
Links:
- added link FL_WHEEL; collision cylinder length=0.02 radius=0.05; visual cylinder length=0.02 radius=0.05
- added link FR_WHEEL; collision cylinder length=0.02 radius=0.05; visual cylinder length=0.02 radius=0.05
- added link RL_WHEEL; collision cylinder length=0.02 radius=0.05; visual cylinder length=0.02 radius=0.05
- added link RR_WHEEL; collision cylinder length=0.02 radius=0.05; visual cylinder length=0.02 radius=0.05
Joints:
- added joint FL_wheel_fixed: type revolute, parent FL_calf, child FL_WHEEL, origin xyz=0 0.035  -0.213 rpy=0 0 0, axis 0 1 0, limit lower=-2147483647 upper=2147483647 effort=20 velocity=10
- added joint FR_wheel_fixed: type revolute, parent FR_calf, child FR_WHEEL, origin xyz=0 -0.035  -0.213 rpy=0 0 0, axis 0 1 0, limit lower=-2147483647 upper=2147483647 effort=20 velocity=10
- added joint RL_wheel_fixed: type revolute, parent RL_calf, child RL_WHEEL, origin xyz=0 0.035  -0.213 rpy=0 0 0, axis 0 1 0, limit lower=-2147483647 upper=2147483647 effort=20 velocity=10
- added joint RR_wheel_fixed: type revolute, parent RR_calf, child RR_WHEEL, origin xyz=0 0.035  -0.213 rpy=0 0 0, axis 0 1 0, limit lower=-2147483647 upper=2147483647 effort=20 velocity=10
